Commit message: added decimals to coordinates

File: body.urdf (robot description, URDF)
Before this commit: robot robot, 2 links, 1 joints
Links:
- link Leg: geometry collision box size=1.0 1.0 1.0; visual box size=1.0 1.0 1.0
- link Torso: geometry collision box size=1.0 1.0 1.0; visual box size=1.0 1.0 1.0

Commit message: did step 37 and now resembles slide 8

File: body.urdf (robot description, URDF)
Before this commit: robot robot, 2 links, 1 joints
Links:
- removed link Leg
- removed link Torso
- added link Link0, mass 1; collision box size=1.0 1.0 1.0; visual box size=1.0 1.0 1.0
- added link Link1, mass 1; collision box size=1.0 1.0 1.0; visual box size=1.0 1.0 1.0
- added link Link2, mass 1; collision box size=1.0 1.0 1.0; visual box size=1.0 1.0 1.0
Joints:
- removed joint Torso_Leg
- added joint Link0_Link1: type revolute, parent Link0, child Link1, origin xyz=0 0 1.0 rpy=0 0 0, axis 0 1 0, limit lower=-3.14159 upper=3.14159 effort=0.0 velocity=0.0
- added joint Link2_Link1: type revolute, parent Link1, child Link2, origin xyz=0 0 1.0 rpy=0 0 0, axis 0 1 0, limit lower=-3.14159 upper=3.14159 effort=0.0 velocity=0.0

Commit message: did step 38 and now resembles slides 9 & 10

File: body.urdf (robot description, URDF)
Before this commit: robot robot, 3 links, 2 joints
Links:
- added link Link3, mass 1; collision box size=1.0 1.0 1.0; visual box size=1.0 1.0 1.0
Joints:
- removed joint Link2_Link1
- added joint Link1_Link2: type revolute, parent Link1, child Link2, origin xyz=0 0 1.0 rpy=0 0 0, axis 0 1 0, limit lower=-3.14159 upper=3.14159 effort=0.0 velocity=0.0
- added joint Link2_Link3: type revolute, parent Link2, child Link3, origin xyz=0 0.5 0.5 rpy=0 0 0, axis 0 1 0, limit lower=-3.14159 upper=3.14159 effort=0.0 velocity=0.0

Commit message: copied slide deck up to step 42

File: body.urdf (robot description, URDF)
Before this commit: robot robot, 4 links, 3 joints
Links:
- added link Link4, mass 1; collision box size=1.0 1.0 1.0; visual box size=1.0 1.0 1.0
- added link Link5, mass 1; collision box size=1.0 1.0 1.0; visual box size=1.0 1.0 1.0
- added link Link6, mass 1; collision box size=1.0 1.0 1.0; visual box size=1.0 1.0 1.0
Joints:
- added joint Link3_Link4: type revolute, parent Link3, child Link4, origin xyz=0 1.0 0 rpy=0 0 0, axis 0 1 0, limit lower=-3.14159 upper=3.14159 effort=0.0 velocity=0.0
- added joint Link4_Link5: type revolute, parent Link4, child Link5, origin xyz=0 0.5 -0.5 rpy=0 0 0, axis 0 1 0, limit lower=-3.14159 upper=3.14159 effort=0.0 velocity=0.0
- added joint Link5_Link6: type revolute, parent Link5, child Link6, origin xyz=0 0 -1 rpy=0 0 0, axis 0 1 0, limit lower=-3.14159 upper=3.14159 effort=0.0 velocity=0.0

Commit message: 3-Link, 2-Joint robot (step 47)

File: body.urdf (robot description, URDF)
Before this commit: robot robot, 7 links, 6 joints
Links:
- removed link Link3
- removed link Link4
- removed link Link5
- removed link Link6
Joints:
- removed joint Link2_Link3
- removed joint Link3_Link4
- removed joint Link4_Link5
- removed joint Link5_Link6
- joint Link0_Link1: origin xyz=0 0 1.0 rpy=0 0 0 -> xyz=1.0 0 1.0 rpy=0 0 0
- joint Link1_Link2: origin xyz=0 0 1.0 rpy=0 0 0 -> xyz=1.0 0 0 rpy=0 0 0

Commit message: changed link names to backleg, torso, and frontleg

File: body.urdf (robot description, URDF)
Before this commit: robot robot, 3 links, 2 joints
Links:
- removed link Link0
- removed link Link1
- removed link Link2
- added link BackLeg, mass 1; collision box size=1.0 1.0 1.0; visual box size=1.0 1.0 1.0
- added link FrontLeg, mass 1; collision box size=1.0 1.0 1.0; visual box size=1.0 1.0 1.0
- added link Torso, mass 1; collision box size=1.0 1.0 1.0; visual box size=1.0 1.0 1.0
Joints:
- removed joint Link0_Link1
- removed joint Link1_Link2
- added joint BackLeg_Torso: type revolute, parent BackLeg, child Torso, origin xyz=1.0 0 1.0 rpy=0 0 0, axis 0 1 0, limit lower=-3.14159 upper=3.14159 effort=0.0 velocity=0.0
- added joint Torso_FrontLeg: type revolute, parent Torso, child FrontLeg, origin xyz=1.0 0 0 rpy=0 0 0, axis 0 1 0, limit lower=-3.14159 upper=3.14159 effort=0.0 velocity=0.0

Commit message: finished up to step 23 in sensor assignment

File: body.urdf (robot description, URDF)
Before this commit: robot robot, 3 links, 2 joints
Joints:
- removed joint BackLeg_Torso
- removed joint Torso_FrontLeg
- added joint FrontLeg_Torso: type revolute, parent FrontLeg, child Torso, origin xyz=1.0 0 1.0 rpy=0 0 0, axis 0 1 0, limit lower=-3.14159 upper=3.14159 effort=0.0 velocity=0.0
- added joint Torso_BackLeg: type revolute, parent Torso, child BackLeg, origin xyz=1.0 0 0 rpy=0 0 0, axis 0 1 0, limit lower=-3.14159 upper=3.14159 effort=0.0 velocity=0.0

Commit message: finished sensors assignment

File: body.urdf (robot description, URDF)
Before this commit: robot robot, 3 links, 2 joints
Joints:
- removed joint FrontLeg_Torso
- added joint Torso_FrontLeg: type revolute, parent Torso, child FrontLeg, origin xyz=2.0 0 1.0 rpy=0 0 0, axis 0 1 0, limit lower=-3.14159 upper=3.14159 effort=0.0 velocity=0.0
- joint Torso_BackLeg: origin xyz=1.0 0 0 rpy=0 0 0 -> xyz=1.0 0 1.0 rpy=0 0 0

Commit message: completed step 18

File: body.urdf (robot description, URDF)
Before this commit: robot robot, 3 links, 2 joints
Links:
- link FrontLeg: geometry collision box size=0.2 1 0.2; visual box size=0.2 1 0.2
Joints:
- joint Torso_FrontLeg: origin xyz=2.0 0 1.0 rpy=0 0 0 -> xyz=0 0.5 1.0 rpy=0 0 0

Commit message: step 22 done

File: body.urdf (robot description, URDF)
Before this commit: robot robot, 3 links, 2 joints
Links:
- link BackLeg: geometry collision box size=0.2 1 0.2; visual box size=0.2 1 0.2
Joints:
- joint Torso_BackLeg: origin xyz=1.0 0 1.0 rpy=0 0 0 -> xyz=0 -0.5 1.0 rpy=0 0 0

Commit message: debugging step 35

File: body.urdf (robot description, URDF)
Before this commit: robot robot, 3 links, 2 joints
Joints:
- joint Torso_BackLeg: axis 0 1 0 -> -1 0 0
- joint Torso_FrontLeg: axis 0 1 0 -> 1 0 0

Commit message: completed step 39

File: body.urdf (robot description, URDF)
Before this commit: robot robot, 3 links, 2 joints
Links:
- added link LeftLeg, mass 1; collision box size=1 0.2 0.2; visual box size=1 0.2 0.2
Joints:
- added joint Torso_LeftLeg: type revolute, parent Torso, child LeftLeg, origin xyz=-0.5 0 1 rpy=0 0 0, axis 1 0 0, limit lower=-3.14159 upper=3.14159 effort=0.0 velocity=0.0
- joint Torso_BackLeg: axis -1 0 0 -> 1 0 0

Commit message: done 40

File: body.urdf (robot description, URDF)
Before this commit: robot robot, 4 links, 3 joints
Links:
- added link RightLeg, mass 1; collision box size=1 0.2 0.2; visual box size=1 0.2 0.2
Joints:
- added joint Torso_RightLeg: type revolute, parent Torso, child RightLeg, origin xyz=0.5 0 1 rpy=0 0 0, axis 1 0 0, limit lower=-3.14159 upper=3.14159 effort=0.0 velocity=0.0

Commit message: done 44

File: body.urdf (robot description, URDF)
Before this commit: robot robot, 5 links, 4 joints
Links:
- added link BackLowerLeg, mass 1; collision box size=0.2 0.2 1; visual box size=0.2 0.2 1
- added link FrontLowerLeg, mass 1; collision box size=0.2 0.2 1; visual box size=0.2 0.2 1
- added link LeftLowerLeg, mass 1; collision box size=0.2 0.2 1; visual box size=0.2 0.2 1
- added link RightLowerLeg, mass 1; collision box size=0.2 0.2 1; visual box size=0.2 0.2 1
Joints:
- added joint BackLeg_BackLowerLeg: type revolute, parent BackLeg, child BackLowerLeg, origin xyz=0 -1 0 rpy=0 0 0, axis 0 0 1, limit lower=-3.14159 upper=3.14159 effort=0.0 velocity=0.0
- added joint FrontLeg_FrontLowerLeg: type revolute, parent FrontLeg, child FrontLowerLeg, origin xyz=0 1 0 rpy=0 0 0, axis 0 0 1, limit lower=-3.14159 upper=3.14159 effort=0.0 velocity=0.0
- added joint LeftLeg_LeftLowerLeg: type revolute, parent LeftLeg, child LeftLowerLeg, origin xyz=-1 0 0 rpy=0 0 0, axis 0 0 1, limit lower=-3.14159 upper=3.14159 effort=0.0 velocity=0.0
- added joint RightLeg_RightLowerLeg: type revolute, parent RightLeg, child RightLowerLeg, origin xyz=1 0 0 rpy=0 0 0, axis 1 0 0, limit lower=-3.14159 upper=3.14159 effort=0.0 velocity=0.0

Commit message: debug

File: body.urdf (robot description, URDF)
Before this commit: robot robot, 9 links, 8 joints
Joints:
- joint RightLeg_RightLowerLeg: axis 1 0 0 -> 0 0 1
- joint Torso_LeftLeg: axis 1 0 0 -> 0 1 0
- joint Torso_RightLeg: axis 1 0 0 -> 0 1 0

Commit message: debugging why children are never better than the parent with numOfGenerations=1

File: body.urdf (robot description, URDF)
Before this commit: robot robot, 9 links, 8 joints
Joints:
- joint BackLeg_BackLowerLeg: axis 0 0 1 -> 1 0 0
- joint FrontLeg_FrontLowerLeg: axis 0 0 1 -> 1 0 0
- joint LeftLeg_LeftLowerLeg: axis 0 0 1 -> 0 1 0
- joint RightLeg_RightLowerLeg: axis 0 0 1 -> 0 1 0

Commit message: quadruped works

File: body.urdf (robot description, URDF)
Before this commit: robot robot, 9 links, 8 joints
Links:
- link RightLeg: geometry collision box size=1 0.1 0.2; visual box size=1 0.1 0.2

Commit message: debug temp

File: body.urdf (robot description, URDF)
Before this commit: robot robot, 9 links, 8 joints
Links:
- added link SecondLeftLeg, mass 1; collision box size=1 0.15 0.15; visual box size=1 0.15 0.15
- added link SecondLeftLowerLeg, mass 1; collision box size=0.15 0.15 1; visual box size=0.15 0.15 1
- added link SecondRightLeg, mass 1; collision box size=1 0.15 0.15; visual box size=1 0.15 0.15
- added link SecondRightLowerLeg, mass 1; collision box size=0.15 0.15 1; visual box size=0.15 0.15 1
- link BackLeg: geometry collision box size=0.15 1 0.15; visual box size=0.15 1 0.15
- link BackLowerLeg: geometry collision box size=0.15 0.15 1; visual box size=0.15 0.15 1
- link FrontLeg: geometry collision box size=0.15 1 0.15; visual box size=0.15 1 0.15
- link FrontLowerLeg: geometry collision box size=0.15 0.15 1; visual box size=0.15 0.15 1
- link LeftLeg: geometry collision box size=1 0.15 0.15; visual box size=1 0.15 0.15
- link LeftLowerLeg: geometry collision box size=0.15 0.15 1; visual box size=0.15 0.15 1
- link RightLeg: geometry collision box size=1 0.15 0.15; visual box size=1 0.15 0.15
- link RightLowerLeg: geometry collision box size=0.15 0.15 1; visual box size=0.15 0.15 1
Joints:
- added joint LeftLeg_SecondLeftLowerLeg: type revolute, parent SecondLeftLeg, child SecondLeftLowerLeg, origin xyz=-1 0 0 rpy=0 0 0, axis 0 1 0, limit lower=-3.14159 upper=3.14159 effort=0.0 velocity=0.0
- added joint RightLeg_SecondRightLowerLeg: type revolute, parent SecondRightLeg, child SecondRightLowerLeg, origin xyz=1 0 0 rpy=0 0 0, axis 0 1 0, limit lower=-3.14159 upper=3.14159 effort=0.0 velocity=0.0
- added joint Torso_SecondLeftLeg: type revolute, parent Torso, child SecondLeftLeg, origin xyz=-0.5 0 1 rpy=0 0 0, axis 0 1 0, limit lower=-3.14159 upper=3.14159 effort=0.0 velocity=0.0
- added joint Torso_SecondRightLeg: type revolute, parent Torso, child SecondRightLeg, origin xyz=0.5 0 1 rpy=0 0 0, axis 0 1 0, limit lower=-3.14159 upper=3.14159 effort=0.0 velocity=0.0

Commit message: hexaped works slowly

File: body.urdf (robot description, URDF)
Before this commit: robot robot, 13 links, 12 joints
Joints:
- removed joint LeftLeg_SecondLeftLowerLeg
- removed joint RightLeg_SecondRightLowerLeg
- added joint SecondLeftLeg_SecondLeftLowerLeg: type revolute, parent SecondLeftLeg, child SecondLeftLowerLeg, origin xyz=-1 0 0 rpy=0 0 0, axis 0 1 0, limit lower=-3.14159 upper=3.14159 effort=0.0 velocity=0.0
- added joint SecondRightLeg_SecondRightLowerLeg: type revolute, parent SecondRightLeg, child SecondRightLowerLeg, origin xyz=1 0 0 rpy=0 0 0, axis 0 1 0, limit lower=-3.14159 upper=3.14159 effort=0.0 velocity=0.0

Commit message: added graphing capability to hexapod

File: body.urdf (robot description, URDF)
Before this commit: robot robot, 9 links, 8 joints
Links:
- added link SecondLeftLeg, mass 1; collision box size=1 0.15 0.15; visual box size=1 0.15 0.15
- added link SecondLeftLowerLeg, mass 1; collision box size=0.15 0.15 1; visual box size=0.15 0.15 1
- added link SecondRightLeg, mass 1; collision box size=1 0.15 0.15; visual box size=1 0.15 0.15
- added link SecondRightLowerLeg, mass 1; collision box size=0.15 0.15 1; visual box size=0.15 0.15 1
- link LeftLeg: geometry collision box size=1 0.15 0.15; visual box size=1 0.15 0.15
- link LeftLowerLeg: geometry collision box size=0.15 0.15 1; visual box size=0.15 0.15 1
- link RightLeg: geometry collision box size=1 0.15 0.15; visual box size=1 0.15 0.15
- link RightLowerLeg: geometry collision box size=0.15 0.15 1; visual box size=0.15 0.15 1
Joints:
- added joint SecondLeftLeg_SecondLeftLowerLeg: type revolute, parent SecondLeftLeg, child SecondLeftLowerLeg, origin xyz=-1 0 0 rpy=0 0 0, axis 0 1 0, limit lower=-3.14159 upper=3.14159 effort=0.0 velocity=0.0
- added joint SecondRightLeg_SecondRightLowerLeg: type revolute, parent SecondRightLeg, child SecondRightLowerLeg, origin xyz=1 0 0 rpy=0 0 0, axis 0 1 0, limit lower=-3.14159 upper=3.14159 effort=0.0 velocity=0.0
- added joint Torso_SecondLeftLeg: type revolute, parent Torso, child SecondLeftLeg, origin xyz=-0.5 0 1 rpy=0 0 0, axis 0 1 0, limit lower=-3.14159 upper=3.14159 effort=0.0 velocity=0.0
- added joint Torso_SecondRightLeg: type revolute, parent Torso, child SecondRightLeg, origin xyz=0.5 0 1 rpy=0 0 0, axis 0 1 0, limit lower=-3.14159 upper=3.14159 effort=0.0 velocity=0.0
